File: PCB/MainSTM_V2/MainSTM_V2.kicad_pcb (KiCad board)
At the start: 2 copper layers, 41 x 38 mm, 39 parts, among them J18 St-Link, J2 St-Link, SW1 SW_Push, U1 LTV-356T, U3 STM32F411RETx, U4 MCP1703A-3302_SOT23, Y1 16MHz

Commit message: STM32 PCB update + BOM
Parts:
- removed J18: St-Link, Connector_PinHeader_2.54mm:PinHeader_1x04_P2.54mm_Horizontal
- added C14: 100nF, Capacitor_SMD:C_0805_2012Metric, B.Cu at (116.8, 85.4)
- added C17: 1uF, Capacitor_SMD:C_0805_2012Metric, F.Cu at (90.5, 103.7)
- added C19: 100nF, Capacitor_SMD:C_0805_2012Metric, F.Cu at (90.5, 101.0)
- added C3: 10uF, Capacitor_Tantalum_SMD:CP_EIA-3216-18_Kemet-A, B.Cu at (114.4, 84.8)
- added CLK: St-Link, Connector_PinHeader_2.54mm:PinHeader_1x04_P2.54mm_Vertical, F.Cu at (119.6, 85.9)
- added D11: Power_On, LED_SMD:LED_1206_3216Metric, F.Cu at (108.0, 82.7)
- added R5: RLed, Resistor_SMD:R_0805_2012Metric, B.Cu at (101.5, 83.5)
- added U2: MIC5205-5.0YM5, Package_TO_SOT_SMD:SOT-23-5, B.Cu at (111.4, 85.2)
- D2: moved to F.Cu
- moved C5 7.27 mm to (103.9, 88.5)
- moved U4 5.97 mm to (100.8, 88.5)
- moved C6 5.50 mm to (97.8, 88.5)
- moved F2 4.07 mm to (112.2, 89.5)
- moved C4 4.06 mm to (106.2, 88.0), turned to 270 degrees
- moved D1 3.00 mm to (108.3, 87.8), turned to 270 degrees
- moved D2 2.10 mm to (101.3, 89.9), turned to 0 degrees
- moved R9 2.06 mm to (99.1, 83.5), turned to 90 degrees
- moved C7 2.04 mm to (104.5, 93.5), turned to 0 degrees
Connections:
- net Net-(C4-Pad1) renamed V_Stable
- C10 pad 1: VDD -> +3V3
- C12 pad 2: VDD -> +3V3
- C6 pad 1: VDD -> +3V3
- C7 pad 2: VDD -> +3V3
- C8 pad 2: VDD -> +3V3
- D2 pad 2: VDD -> +3V3
- J2 pad 1: GND -> +3V3
- R2 pad 1: VDD -> +3V3
- U3 pad 1: VDD -> +3V3
- U3 pad 13: VDD -> +3V3
- U3 pad 19: VDD -> +3V3
- U3 pad 32: VDD -> +3V3
- U3 pad 48: VDD -> +3V3
- U3 pad 64: VDD -> +3V3
- U4 pad 2: VDD -> +3V3
Routing:
- net +3V3: track 0.00 -> 103.0 mm, vias 0 -> 6
- net VDD: track 80.2 -> 0.00 mm, vias 5 -> 0
- net +5V: track 113.1 -> 130.6 mm, vias 1 -> 4
- net Net-(D11-Pad1): track 0.00 -> 6.42 mm, vias 0 -> 1
- net Net-(D2-Pad1): track 2.77 -> 6.40 mm, vias 0 -> 1
- net V_Stable: track 16.8 -> 13.7 mm
- net RESET: track 81.0 -> 77.9 mm
- net GND: track 12.3 -> 9.40 mm, vias 5 -> 8
- net SWD_IO: track 22.0 -> 24.0 mm
- net SWD_CLK: track 22.1 -> 20.5 mm
- net VPP: track 6.03 -> 4.78 mm
- net Net-(D1-Pad2): track 3.56 -> 2.82 mm
Other:
- board text added: "G"
- board text added: "IO"
- board text added: "RST"
